File: power.kicad_sch (KiCad schematic)
At the start: 12 parts, among them J2 S2B-PH-SM4-TB(LF)(SN), U2 MCP73832-2-OT, U4 LM66200DRLR

Commit message: Update schematic
Parts:
- added R18: k, symbol Device:R
Connections:
- net +BATT: now also R18.2
- net at U4.8 (ST): now also R18.1
Other:
- note added: "sidenote: we might need to swap VIN1 & VIN2 between +BATT & VBUS due to 4.7v vs 5v"
Changed lines of the file:
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@@
+		)
+	)
+	(text "sidenote: we might need to swap\nVIN1 & VIN2 between +BATT & VBUS due to 4.7v vs 5v"
+		(exclude_from_sim no)
+		(at 159.766 88.138 0)
+		(effects
+			(font
+				(size 1.27 1.27)
+			)
+			(justify left)
 		)
 	)
@@
 	)
 	(junction
+		(at 233.68 43.18)
+		(diameter 0)
+		(color 0 0 0 0)
+	)
+	(junction
 		(at 83.82 35.56)
 		(diameter 0)
@@
 	(wire
 		(pts
+			(xy 233.68 41.91) (xy 233.68 43.18)
+		)
+		(stroke
+			(width 0)
+			(type default)
+		)
+	)
+	(wire
+		(pts
 			(xy 53.34 175.26) (xy 53.34 173.99)
 		)
@@
 		(pts
 			(xy 95.25 35.56) (xy 101.6 35.56)
+		)
+		(stroke
+			(width 0)
+			(type default)
+		)
+	)
+	(wire
+		(pts
+			(xy 233.68 31.75) (xy 233.68 34.29)
 		)
 		(stroke
@@
 	)
 	(symbol
+		(lib_id "power:+BATT")
+		(at 233.68 31.75 0)
+		(unit 1)
+		(exclude_from_sim no)
+		(in_bom yes)
+		(on_board yes)
+		(dnp no)
+		(fields_autoplaced yes)
+		(property "Reference" "#PWR036"
+			(at 233.68 35.56 0)
+			(effects
+				(font
+					(size 1.27 1.27)
+				)
+				(hide yes)
+			)
+		)
+		(property "Value" "+BATT"
+			(at 233.68 26.67 0)
+			(effects
+				(font
+					(size 1.27 1.27)
+				)
+			)
+		)
+		(property "Footprint" ""
+			(at 233.68 31.75 0)
+			(effects
+				(font
+					(size 1.27 1.27)
+				)
+				(hide yes)
+			)
+		)
+		(property "Datasheet" ""
+			(at 233.68 31.75 0)
+			(effects
+				(font
+					(size 1.27 1.27)
+				)
+				(hide yes)
+			)
+		)
+		(property "Description" "Power symbol creates a global label with name \"+BATT\""
+			(at 233.68 31.75 0)
+			(effects
+				(font
+					(size 1.27 1.27)
+				)
+				(hide yes)
+			)
+		)
+		(pin "1"
+		)
+		(instances
+			(project "siiren"
+				(path "/f2af4cd4-99cf-4d01-92f6-6413371e0fe3/8a3d119c-67dd-4f4a-8377-40fc3a7c71aa"
+					(reference "#PWR036")
+					(unit 1)
+				)
+			)
+		)
+	)
+	(symbol
 		(lib_id "power:+3.3V")
 		(at 121.92 50.8 0)
@@
 	(symbol
 		(lib_id "power:GND")
-		(at 139.7 133.35 0)
+		(at 144.78 133.35 0)
 		(unit 1)
 		(exclude_from_sim no)
@@
 		(fields_autoplaced yes)
 		(property "Reference" "#PWR035"
-			(at 139.7 139.7 0)
+			(at 144.78 139.7 0)
 			(effects
 				(font
@@
 		)
 		(property "Value" "GND"
-			(at 139.7 138.43 0)
+			(at 144.78 138.43 0)
 			(effects
 				(font
@@
 		)
 		(property "Footprint" ""
-			(at 139.7 133.35 0)
+			(at 144.78 133.35 0)
 			(effects
 				(font
@@
 		)
 		(property "Datasheet" ""
-			(at 139.7 133.35 0)
+			(at 144.78 133.35 0)
 			(effects
 				(font
@@
 		)
 		(property "Description" "Power symbol creates a global label with name \"GND\" , ground"
-			(at 139.7 133.35 0)
+			(at 144.78 133.35 0)
 			(effects
 				(font
@@
 					(unit 1)
 				)
+			)
+		)
+	)
+	(symbol
+		(lib_id "Device:R")
+		(at 233.68 38.1 180)
+		(unit 1)
+		(exclude_from_sim no)
+		(in_bom yes)
+		(on_board yes)
+		(dnp no)
+		(fields_autoplaced yes)
+		(property "Reference" "R18"
+			(at 236.22 36.8299 0)
+			(effects
+				(font
+					(size 1.27 1.27)
+				)
+				(justify right)
+			)
+		)
+		(property "Value" "k"
+			(at 236.22 39.3699 0)
+			(effects
+				(font
+					(size 1.27 1.27)
+				)
+				(justify right)
+			)
+		)
+		(property "Footprint" ""
+			(at 235.458 38.1 90)
+			(effects
+				(font
+					(size 1.27 1.27)
+				)
+				(hide yes)
+			)
+		)
+		(property "Datasheet" "~"
+			(at 233.68 38.1 0)
+			(effects
+				(font
+					(size 1.27 1.27)
+				)
+				(hide yes)
+			)
+		)
+		(property "Description" "Resistor"
+			(at 233.68 38.1 0)
+			(effects
+				(font
+					(size 1.27 1.27)
+				)
+				(hide yes)
+			)
+		)
+		(pin "1"
+		)
+		(pin "2"
+		)
+		(instances
+			(project "siiren"
+				(path "/f2af4cd4-99cf-4d01-92f6-6413371e0fe3/8a3d119c-67dd-4f4a-8377-40fc3a7c71aa"
+					(reference "R18")
+					(unit 1)
+				)
