File: siiren.kicad_pcb (KiCad board)
At the start: 2 copper layers, 60 x 30 mm, 14 parts, among them J1 USB_C_Receptacle_USB2.0_16P, J2 S2B-PH-SM4-TB(LF)(SN), SW2 K1-1210UN-01, U1 ESP32-C3-WROOM-02, U2 MCP73832-2-OT, U3 USBLC6-2SC6

Commit message: Update schematic
Parts:
- moved J2 51.8 mm to (84.0, 35.2), turned to -90 degrees
- moved D1 11.0 mm to (59.5, 50.5)
- moved D4 11.0 mm to (59.7, 53.5)
- moved U2 9.24 mm to (67.5, 54.0)
- moved R5 9.07 mm to (70.8, 48.8)
- moved R3 9.03 mm to (51.8, 54.4), turned to 180 degrees
- moved R4 4.23 mm to (55.0, 54.4), turned to 0 degrees
- moved U3 4.09 mm to (72.5, 53.6)
- moved SW2 3.33 mm to (77.8, 46.0)
- moved R6 3.21 mm to (79.2, 48.4)
- moved R1 1.76 mm to (79.1, 54.6)
- moved R2 1.76 mm to (79.1, 52.9)
- moved J1 0.77 mm to (87.0, 54.0)
Routing:
- net +BATT: track 41.8 -> 0.00 mm
- net unconnected-(U1-IO2-Pad16): track 37.9 -> 0.00 mm
- net /USB/USB_D-_RAW: track 8.19 -> 0.00 mm
- net /USB/USB_D+_RAW: track 5.12 -> 0.00 mm
- net VBUS: track 0.00 -> 2.83 mm
- net /USB/USB_DN: track 2.29 -> 0.00 mm
- net /USB/USB_DP: track 2.23 -> 0.00 mm
- net GND: track 1.11 -> 0.00 mm, vias 1 -> 0
